File: hw/AS5055A.sch (KiCad schematic (older format))
At the start: 8 parts, among them U2 TXB0108, U3 AS5055A

Commit message: added missed save
Parts:
- removed JP1: JUMPER, symbol JUMPER
Connections:
- wire segments 51 -> 47
- no-connect marks 8 -> 10
Changed lines of the file:
@@
-	1    0    0    -1
-$EndComp
-Wire Wire Line
-	5650 4200 5650 4350
-Wire Wire Line
-	5900 4200 5650 4200
-Connection ~ 5650 4200
-$Comp
-L GND #PWR020
-U 1 1 53875085
-P 5650 4350
-F 0 "#PWR020" H 5650 4350 30  0001 C CNN
-F 1 "GND" H 5650 4280 30  0001 C CNN
-F 2 "" H 5650 4350 60  0000 C CNN
-F 3 "" H 5650 4350 60  0000 C CNN
-	1    5650 4350
 	1    0    0    -1
 $EndComp
@@
 $EndComp
 NoConn ~ 5900 4800
-Wire Wire Line
-	5900 4300 5650 4300
-Connection ~ 5650 4300
 Wire Wire Line
 	7350 4700 7650 4700
@@
 	8350 3550 8350 3650
 Connection ~ 8350 3600
-$Comp
-L JUMPER JP1
-U 1 1 5387C86C
-P 5500 4100
-F 0 "JP1" H 5500 4250 60  0000 C CNN
-F 1 "JUMPER" H 5500 4020 40  0000 C CNN
-F 2 "" H 5500 4100 60  0000 C CNN
-F 3 "" H 5500 4100 60  0000 C CNN
-	1    5500 4100
-	1    0    0    -1
-$EndComp
-Wire Wire Line
-	5900 4100 5800 4100
-Wire Wire Line
-	5200 4100 5150 4100
-Wire Wire Line
-	5150 4100 5150 4150
-$Comp
-L GND #PWR023
-U 1 1 5387C9CE
-P 5150 4150
-F 0 "#PWR023" H 5150 4150 30  0001 C CNN
-F 1 "GND" H 5150 4080 30  0001 C CNN
-F 2 "" H 5150 4150 60  0000 C CNN
-F 3 "" H 5150 4150 60  0000 C CNN
-	1    5150 4150
-	1    0    0    -1
-$EndComp
 Text HLabel 10250 4150 0    60   Input ~ 0
 MOSI
@@
 Text Label 10350 4650 0    60   ~ 0
 INT_B
+NoConn ~ 6550 5150
+Wire Wire Line
+	5900 4300 5450 4300
+Wire Wire Line
+	5450 4200 5450 4400
 $Comp
-L GND #PWR024
-U 1 1 53A54204
-P 6550 5200
-F 0 "#PWR024" H 6550 5200 30  0001 C CNN
-F 1 "GND" H 6550 5130 30  0001 C CNN
-F 2 "" H 6550 5200 60  0000 C CNN
-F 3 "" H 6550 5200 60  0000 C CNN
-	1    6550 5200
+L GND #PWR?
+U 1 1 53C2438D
+P 5450 4400
+F 0 "#PWR?" H 5450 4400 30  0001 C CNN
+F 1 "GND" H 5450 4330 30  0001 C CNN
+F 2 "" H 5450 4400 60  0000 C CNN
+F 3 "" H 5450 4400 60  0000 C CNN
+	1    5450 4400
 	1    0    0    -1
 $EndComp
+NoConn ~ 5900 4100
 Wire Wire Line
-	6550 5200 6550 5150
+	5900 4200 5450 4200
+Connection ~ 5450 4300
 $EndSCHEMATC
